Commit message: separated hrp2 and hyq in two different packages

File: data/hrp2/urdf/hrp2_larm_rom.urdf (robot description, URDF)
Before this commit: robot hrp2_trunk_flexible, 6 links, 5 joints
Links:
- link BODY: geometry 
- link HEAD_LINK0: geometry 
- link HEAD_LINK1: geometry 
- link torso: geometry collision mesh filename=package://hrp2-rbprm/meshes/hrp2_larm_rom.stl; visual mesh filename=package://hrp2-rbprm/meshes/hrp2_larm_rom.stl

File: data/hrp2/urdf/hrp2_lleg_rom.urdf (robot description, URDF)
Before this commit: robot hrp2_rleg_rom, 6 links, 5 joints
Links:
- link BODY: geometry collision mesh filename=package://hrp2-rbprm/meshes/hrp2_lleg_rom.stl; visual mesh filename=package://hrp2-rbprm/meshes/hrp2_lleg_rom.stl

File: data/hrp2/urdf/hrp2_rarm_rom.urdf (robot description, URDF)
Before this commit: robot hrp2_larm_rom, 6 links, 5 joints
Links:
- link torso: geometry collision mesh filename=package://hrp2-rbprm/meshes/hrp2_rarm_rom.stl; visual mesh filename=package://hrp2-rbprm/meshes/hrp2_rarm_rom.stl

File: data/hrp2/urdf/hrp2_rleg_rom.urdf (robot description, URDF)
Before this commit: robot hrp2_rarm_rom, 6 links, 5 joints
Links:
- link BODY: geometry collision mesh filename=package://hrp2-rbprm/meshes/hrp2_rleg_rom.stl; visual mesh filename=package://hrp2-rbprm/meshes/hrp2_rleg_rom.stl
- link torso: geometry 

File: data/hrp2/urdf/hrp2_rom.urdf (robot description, URDF)
Before this commit: robot hrp2_trunk08, 1 links, 0 joints
Links:
- link base_link: geometry collision mesh filename=package://hrp2-rbprm/meshes/hrp2_rom.stl; visual mesh filename=package://hrp2-rbprm/meshes/hrp2_rom.stl

File: data/hrp2/urdf/hrp2_trunk.urdf (robot description, URDF)
Before this commit: robot hrp2_rom, 1 links, 0 joints
Links:
- link base_link: geometry collision mesh filename=package://hrp2-rbprm/meshes/hrp2_trunk.stl; visual mesh filename=package://hrp2-rbprm/meshes/hrp2_trunk.stl

File: data/hrp2/urdf/hrp2_trunk08.urdf (robot description, URDF)
Before this commit: robot hrp2_trunk, 1 links, 0 joints
Links:
- link base_link: geometry collision mesh filename=package://hrp2-rbprm/meshes/hrp2_trunk08.stl; visual mesh filename=package://hrp2-rbprm/meshes/hrp2_trunk08.stl

File: data/hrp2/urdf/hrp2_trunk_flexible.urdf (robot description, URDF)
Before this commit: robot hrp2_lleg_rom, 6 links, 5 joints
Links:
- link BODY: geometry collision mesh filename=package://hrp2-rbprm/meshes/hrp2_trunk_body.stl; visual mesh filename=package://hrp2-rbprm/meshes/hrp2_trunk_body_view.dae
- link HEAD_LINK0: geometry collision mesh filename=package://hrp2_14_description/meshes/convex/HEAD_LINK0.dae; visual mesh filename=package://hrp2_14_description/meshes/HEAD_LINK0.dae
- link HEAD_LINK1: geometry collision mesh filename=package://hrp2_14_description/meshes/convex/HEAD_LINK1.dae; visual mesh filename=package://hrp2_14_description/meshes/HEAD_LINK1.dae
- link torso: geometry collision mesh filename=package://hrp2-rbprm/meshes/hrp2_trunk_torso.stl; visual mesh filename=package://hrp2-rbprm/meshes/hrp2_trunk_torso_view.dae

File: data/hyq/urdf/hyq_lfleg_rom.urdf (robot description, URDF)
Before this commit: robot hyq_trunk_large, 1 links, 0 joints
Links:
- link base_link: geometry collision mesh filename=package://hyq-rbprm/meshes/hyq/hyq_lfleg_rom.stl; visual mesh filename=package://hyq-rbprm/meshes/hyq/hyq_lfleg_rom.stl

File: data/hyq/urdf/hyq_lhleg_rom.urdf (robot description, URDF)
Before this commit: robot hyq_rhleg_rom, 1 links, 0 joints
Links:
- link base_link: geometry collision mesh filename=package://hyq-rbprm/meshes/hyq/hyq_lhleg_rom.stl; visual mesh filename=package://hyq-rbprm/meshes/hyq/hyq_lhleg_rom.stl

File: data/hyq/urdf/hyq_rfleg_rom.urdf (robot description, URDF)
Before this commit: robot hyq_rom, 1 links, 0 joints
Links:
- link base_link: geometry collision mesh filename=package://hyq-rbprm/meshes/hyq/hyq_rfleg_rom.stl; visual mesh filename=package://hyq-rbprm/meshes/hyq/hyq_rfleg_rom.stl

File: data/hyq/urdf/hyq_rhleg_rom.urdf (robot description, URDF)
Before this commit: robot hyq_rfleg_rom, 1 links, 0 joints
Links:
- link base_link: geometry collision mesh filename=package://hyq-rbprm/meshes/hyq/hyq_rhleg_rom.stl; visual mesh filename=package://hyq-rbprm/meshes/hyq/hyq_rhleg_rom.stl

File: data/hyq/urdf/hyq_rom.urdf (robot description, URDF)
Before this commit: robot hyq_lfleg_rom, 1 links, 0 joints
Links:
- link base_link: geometry collision mesh filename=package://hyq-rbprm/meshes/hyq/hyq_rom.stl; visual mesh filename=package://hyq-rbprm/meshes/hyq/hyq_rom.stl

File: data/hyq/urdf/hyq_trunk.urdf (robot description, URDF)
Before this commit: robot hyq_trunk, 1 links, 0 joints
Links:
- link base_link: geometry collision mesh filename=package://hyq-rbprm/meshes/hyq/hyq_trunk.stl; visual mesh filename=package://hyq-rbprm/meshes/hyq/hyq_all.stl

File: data/hyq/urdf/hyq_trunk_large.urdf (robot description, URDF)
Before this commit: robot hyq_lhleg_rom, 1 links, 0 joints
Links:
- link base_link: geometry collision mesh filename=package://hyq-rbprm/meshes/hyq/hyq_trunk_large.stl; visual mesh filename=package://hyq-rbprm/meshes/hyq/hyq_all.stl
