Commit message: add files for Talos

File: data/talos/urdf/talos_larm_rom.urdf (robot description, URDF)
Before this commit: robot talos_larm_rom, 5 links, 4 joints
Links:
- removed link head_1_link
- removed link head_2_link
- link torso_2_link: geometry collision mesh filename=package://talos-rbprm/meshes/talos_larm_rom.stl scale=1 1 1; visual mesh filename=package://talos-rbprm/meshes/talos_larm_rom.dae scale=1 1 1
Joints:
- removed joint head_1_joint
- removed joint head_2_joint
- joint torso_1_joint: limit lower=-1.308996939 upper=1.308996939 effort=78.0 velocity=5.4 -> lower=-1.25663706144 upper=1.25663706144 effort=78.0 velocity=5.4
- joint torso_2_joint: limit lower=-0.261799387799 upper=0.785398163397 effort=78.0 velocity=5.4 -> lower=-0.226892802759 upper=0.733038285838 effort=78.0 velocity=5.4

File: data/talos/urdf/talos_lleg_rom.urdf (robot description, URDF)
Before this commit: robot talos_lleg_rom, 5 links, 4 joints
Links:
- removed link head_1_link
- removed link head_2_link
- link base_link: geometry collision mesh filename=package://talos-rbprm/meshes/talos_lleg_rom.stl scale=1 1 1; visual mesh filename=package://talos-rbprm/meshes/talos_lleg_rom.dae scale=1 1 1
Joints:
- removed joint head_1_joint
- removed joint head_2_joint
- joint torso_1_joint: limit lower=-1.308996939 upper=1.308996939 effort=78.0 velocity=5.4 -> lower=-1.25663706144 upper=1.25663706144 effort=78.0 velocity=5.4
- joint torso_2_joint: limit lower=-0.261799387799 upper=0.785398163397 effort=78.0 velocity=5.4 -> lower=-0.226892802759 upper=0.733038285838 effort=78.0 velocity=5.4

File: data/talos/urdf/talos_rarm_rom.urdf (robot description, URDF)
Before this commit: robot talos_rarm_rom, 5 links, 4 joints
Links:
- removed link head_1_link
- removed link head_2_link
- link torso_2_link: geometry collision mesh filename=package://talos-rbprm/meshes/talos_rarm_rom.stl scale=1 1 1; visual mesh filename=package://talos-rbprm/meshes/talos_rarm_rom.dae scale=1 1 1
Joints:
- removed joint head_1_joint
- removed joint head_2_joint
- joint torso_1_joint: limit lower=-1.308996939 upper=1.308996939 effort=78.0 velocity=5.4 -> lower=-1.25663706144 upper=1.25663706144 effort=78.0 velocity=5.4
- joint torso_2_joint: limit lower=-0.261799387799 upper=0.785398163397 effort=78.0 velocity=5.4 -> lower=-0.226892802759 upper=0.733038285838 effort=78.0 velocity=5.4

File: data/talos/urdf/talos_rleg_rom.urdf (robot description, URDF)
Before this commit: robot talos_rleg_rom, 5 links, 4 joints
Links:
- removed link head_1_link
- removed link head_2_link
- link base_link: geometry collision mesh filename=package://talos-rbprm/meshes/talos_rleg_rom.stl scale=1 1 1; visual mesh filename=package://talos-rbprm/meshes/talos_rleg_rom.dae scale=1 1 1
Joints:
- removed joint head_1_joint
- removed joint head_2_joint
- joint torso_1_joint: limit lower=-1.308996939 upper=1.308996939 effort=78.0 velocity=5.4 -> lower=-1.25663706144 upper=1.25663706144 effort=78.0 velocity=5.4
- joint torso_2_joint: limit lower=-0.261799387799 upper=0.785398163397 effort=78.0 velocity=5.4 -> lower=-0.226892802759 upper=0.733038285838 effort=78.0 velocity=5.4

File: data/talos/urdf/talos_trunk.urdf (robot description, URDF)
Before this commit: robot talos_trunk, 5 links, 4 joints
Links:
- removed link head_1_link
- removed link head_2_link
- link base_link: geometry collision mesh filename=package://talos-rbprm/meshes/talos_trunk_lower.stl scale=1 1 1; visual mesh filename=package://talos-rbprm/meshes/talos_trunk_lower_visual.dae scale=1 1 1
- link torso_1_link: geometry 
- link torso_2_link: geometry collision mesh filename=package://talos-rbprm/meshes/talos_trunk_upper.stl scale=1 1 1; visual mesh filename=package://talos-rbprm/meshes/talos_trunk_upper_visual.dae scale=1 1 1
Joints:
- removed joint head_1_joint
- removed joint head_2_joint
- joint torso_1_joint: limit lower=-1.308996939 upper=1.308996939 effort=78.0 velocity=5.4 -> lower=-1.25663706144 upper=1.25663706144 effort=78.0 velocity=5.4
- joint torso_2_joint: limit lower=-0.261799387799 upper=0.785398163397 effort=78.0 velocity=5.4 -> lower=-0.226892802759 upper=0.733038285838 effort=78.0 velocity=5.4
