Commit message: update hyq data

File: data/hyq/urdf/hyq_lhleg_rom.urdf (robot description, URDF)
Before this commit: robot hyq_lhleg_rom, 1 links, 0 joints
Links:
- removed link base_link
- added link hyq_lhleg_link; collision mesh filename=package://hyq-rbprm/meshes/hyq_lhleg_rom.stl; visual mesh filename=package://hyq-rbprm/meshes/hyq_lhleg_rom.stl

File: data/hyq/urdf/hyq_rfleg_rom.urdf (robot description, URDF)
Before this commit: robot hyq_rfleg_rom, 1 links, 0 joints
Links:
- removed link base_link
- added link hyq_rfleg_link; collision mesh filename=package://hyq-rbprm/meshes/hyq_rfleg_rom.stl; visual mesh filename=package://hyq-rbprm/meshes/hyq_rfleg_rom.stl

File: data/hyq/urdf/hyq_rhleg_rom.urdf (robot description, URDF)
Before this commit: robot hyq_rhleg_rom, 1 links, 0 joints
Links:
- removed link base_link
- added link hyq_rhleg_link; collision mesh filename=package://hyq-rbprm/meshes/hyq_rhleg_rom.stl; visual mesh filename=package://hyq-rbprm/meshes/hyq_rhleg_rom.stl

File: data/hyq/urdf/hyq_rom.urdf (robot description, URDF)
Before this commit: robot hyq_rom, 1 links, 0 joints
Links:
- link base_link: geometry collision mesh filename=package://hyq-rbprm/meshes/hyq_rom.stl; visual mesh filename=package://hyq-rbprm/meshes/hyq_rom.stl

File: data/hyq/urdf/hyq_trunk.urdf (robot description, URDF)
Before this commit: robot hyq_trunk, 1 links, 0 joints
Links:
- link base_link: geometry collision mesh filename=package://hyq-rbprm/meshes/hyq_trunk.stl; visual mesh filename=package://hyq-rbprm/meshes/hyq_all.stl

File: data/hyq/urdf/hyq_trunk_large.urdf (robot description, URDF)
Before this commit: robot hyq_trunk_large, 1 links, 0 joints
Links:
- link base_link: geometry collision mesh filename=package://hyq-rbprm/meshes/hyq_trunk_large.stl; visual mesh filename=package://hyq-rbprm/meshes/hyq_all.stl

File: data/hyq/urdf/hyq_trunk_large_realist.urdf (robot description, URDF)
Before this commit: robot hyq_lfleg_rom, 1 links, 0 joints
Links:
- removed link hyq_lfleg_link
- added link base_link; collision mesh filename=package://hyq-rbprm/meshes/hyq_trunk_large.stl; visual mesh filename=package://hyq-rbprm/meshes/hyq_all_realist.stl
