Commit message: hyq_abstract : add a dae with color and transparency for ROMs

File: data/hyq/urdf/hyq_trunk_large.urdf (robot description, URDF)
Before this commit: robot hyq_trunk_large, 1 links, 0 joints
Links:
- link base_link: geometry collision mesh filename=package://hyq-rbprm/meshes/hyq_trunk_large.stl; visual mesh filename=package://hyq-rbprm/meshes/hyq_visual.dae
