Commit message: [hyq] change abstract mass to correspond to fullBody

File: data/hyq/urdf/hyq_trunk.urdf (robot description, URDF)
Before this commit: robot hyq_trunk, 1 links, 0 joints
Links:
- link base_link: mass 50.26 -> 76.07

File: data/hyq/urdf/hyq_trunk_large.urdf (robot description, URDF)
Before this commit: robot hyq_trunk_large, 1 links, 0 joints
Links:
- link base_link: mass 50.26 -> 76.07
